File: KiCad_Project/wiringharness2021/wiringharness2021.sch (KiCad schematic (older format))
At the start: 0 parts

Commit message: Significant progress on schematic. Added more modules
Parts:
- added BT?: 12v Battery, symbol Device:Battery
- added BZ? (x4): Fuel Injector, symbol Device:Buzzer
- added D?: LED, symbol Device:LED
- added E? (x4): Spark Plug, symbol Device:SPARK_GAP
- added F?: 100A Fuse, symbol Device:Fuse
- added M? (x2): Fuel Pump, symbol Motor:Motor_DC
- added SW? (x4): MAIN SHUTOFF, symbol Switch:SW_DIP_x01
- added SW?: UPSHIFT, symbol Switch:SW_DIP_x01
- added SW?: DOWNSHIFT, symbol Switch:SW_DIP_x01
- added SW?: NEUTRAL, symbol Switch:SW_DIP_x01
- added SW?: START, symbol Switch:SW_DIP_x01
- added T? (x4): Coil Pack, symbol Device:Transformer_1P_1S
- added U?: MXS1.2, symbol harnesslib:AIMMXL
- added U?: BOSCH_W0133-1605554, symbol harnesslib:BOSCH_W0133-1605554
- added U?: BSPD, symbol harnesslib:BSPD
- added U?: Haltech Connector A, symbol harnesslib:HaltechElite1500A
- added U?: Haltech Connector B, symbol harnesslib:HaltechElite1500B
- added U?: PMU16DL, symbol harnesslib:PMU16DL
- added U?: 91CP16-3 Pressure Sensor, symbol harnesslib:91CP16-3
- added U?: WirelessTelemetry, symbol harnesslib:WirelessTelemetry
- added U?: Shift Controller, symbol harnesslib:WirelessTelemetry
- added U?: Oil Pressure Sensor, symbol harnesslib:91CP16-3
- added U?: Coolant Temp Sensor, symbol harnesslib:91CP16-3
- added U?: Crank Position Sensor, symbol harnesslib:91CP16-3
- added U?: Cam Position Sensor, symbol harnesslib:91CP16-3
Connections:
- new net: T?.2 (AB), U?.6 (OUT1)
- new net: T?.2 (AB), U?.7 (OUT2)
- new net: T?.2 (AB), U?.8 (OUT3)
- new net: T?.2 (AB), U?.9 (OUT4)
- new net: F?.1, SW?.1
- new net: BT?.1 (+), F?.2
- new net: E?.2, T?.3 (SA) (x4)
- new net: E?.1, T?.4 (SB) (x4)
- new net +12v: SW?.2, U?.0 (+12v_SUPPLY), U?.13 (+Vbattery), U?.3 (+Vbattery), U?.5 (+12v), U?.8 (+Vbattery)
- new net CANH: U?.11 (CANH), U?.11 (CANH), U?.23 (CAN1H), U?.23 (CANH)
- new net CANL: U?.12 (CANL), U?.12 (CANL), U?.24 (CANL), U?.36 (CAN1L)
- new net COIL1: U?.1 (IN1), U?.3 (IGNITION#1)
- new net COIL2: U?.2 (IN2), U?.4 (IGNITION#2)
- new net COIL3: U?.3 (IN3), U?.5 (IGNITION#3)
- new net COIL4: U?.4 (IN4), U?.6 (IGNITION#4)
- new net COILPACK_SUPPLY: T?.1 (AA), T?.1 (AA), T?.1 (AA), T?.1 (AA), U?.13 (O4)
- new net FUELPRES: U?.2 (OUT)
- new net FUELPUMP_SUPPLY: M?.1 (+)
- new net GND: BT?.2 (-), M?.2 (-), U?.1 (GND), U?.10 (GND), U?.11 (GND), U?.12 (GND), U?.14 (GND), U?.15 (GND), U?.16 (GND), U?.16 (GND), U?.2 (GND), U?.2 (GND), U?.25 (Ground), U?.5 (GND), U?.6 (GND)
- new net INJ1: BZ?.1 (-), U?.19 (INJECTOR#1)
- new net INJ2: BZ?.1 (-), U?.20 (INJECTOR#2)
- new net INJ3: BZ?.1 (-), U?.21 (INJECTOR#3)
- new net INJ4: BZ?.1 (-), U?.22 (INJECTOR#4)
- new net INJ_SUPPLY: BZ?.2 (+), BZ?.2 (+), BZ?.2 (+), BZ?.2 (+), U?.26 (ECU_Injector_Power_Input), U?.39 (O2)
Other:
- note added: "Battery"
- note added: "Dash"
- note added: "ENGINE"
- note added: "Fuel"
- note added: "Haltech Elite 1500 ECU"
- note added: "Ignition"
- note added: "Steering Wheel"
