File: KiCad_Project/wiringharness2021/wiringharness2021.sch (KiCad schematic (older format))
At the start: 53 parts, among them M1 Water Pump, M2 Starter Motor, M3 FAN, M4 FAN, M5 Fuel Pump, SW1 UPSHIFT, SW2 DOWNSHIFT, SW3 NEUTRAL, SW4 START, SW5 BRAKE OVERTRAVEL, SW6 DRIVER KILL, SW7 MAIN SHUTOFF, T1 Coil Pack, T2 Coil Pack, T3 Coil Pack, T4 Coil Pack, U1 HaltechElite1500_CONA, U10 Cam Position, U11 Crank Position, U12 WirelessTelemetry, U13 Accel. Pedal Pos 1, U14 BOSCH_280750149, U15 ShiftController, U16 Accel. Pedal Pos 2, U17 Brake Pressure, U18 BSPD, U19 AIM_MXS1.2, U2 HaltechElite1500_CONB, U20 Fuel Pressure Sensor, U3 PMU16DL, U4 Oil Pres., U5 Coolant Temp, U6 Air Temp, U7 BOSCH_W0133-1605554, U8 Knock Sensor, U9 Air Pressure

Commit message: Touch ups and re-export
Parts:
- T1: value Coil Pack -> Coil Pack 1
- T2: value Coil Pack -> Coil Pack 2
- T3: value Coil Pack -> Coil Pack 3
- T4: value Coil Pack -> Coil Pack 4
Connections:
- wire segments 46 -> 49
Other:
- moved on the sheet: D1, R1, SW1, SW2, SW3, SW4
Changed lines of the file:
@@
 U 1 1 6013A0A1
 P 11050 1250
-F 0 "BT1" H 11150 1250 50  0000 L CNN
-F 1 "12v Battery" H 11150 1150 50  0000 L CNN
+F 0 "BT1" H 11150 1250 50  0001 L CNN
+F 1 "12v Battery" H 11150 1200 50  0000 L CNN
 F 2 "" V 11050 1310 50  0001 C CNN
 F 3 "~" V 11050 1310 50  0001 C CNN
@@
 U 1 1 60142DCD
 P 10750 1050
-F 0 "F1" V 10553 1050 50  0000 C CNN
+F 0 "F1" V 10553 1050 50  0001 C CNN
 F 1 "100A Fuse" V 10644 1050 50  0000 C CNN
 F 2 "" V 10680 1050 50  0001 C CNN
@@
 Wire Wire Line
 	10600 1050 10500 1050
-Text Notes 10300 700  0    50   ~ 0
+Text Notes 10300 550  0    50   ~ 0
 Battery
 Text GLabel 1850 5450 2    50   Input ~ 0
@@
 L power:GND #PWR010
 U 1 1 60150D47
-P 5000 1700
-F 0 "#PWR010" H 5000 1450 50  0001 C CNN
-F 1 "GND" H 5000 1550 50  0000 C CNN
-F 2 "" H 5000 1700 50  0001 C CNN
-F 3 "" H 5000 1700 50  0001 C CNN
-	1    5000 1700
+P 4950 1900
+F 0 "#PWR010" H 4950 1650 50  0001 C CNN
+F 1 "GND" H 4950 1750 50  0000 C CNN
+F 2 "" H 4950 1900 50  0001 C CNN
+F 3 "" H 4950 1900 50  0001 C CNN
+	1    4950 1900
 	1    0    0    -1
 $EndComp
@@
 U 1 1 60158480
 P 4450 5450
-F 0 "T1" H 4450 5831 50  0000 C CNN
-F 1 "Coil Pack" H 4450 5740 50  0000 C CNN
+F 0 "T1" H 4450 5831 50  0001 C CNN
+F 1 "Coil Pack 1" H 4450 5740 50  0000 C CNN
 F 2 "" H 4450 5450 50  0001 C CNN
 F 3 "~" H 4450 5450 50  0001 C CNN
@@
 U 1 1 6016BA0D
 P 4450 6100
-F 0 "T2" H 4450 6481 50  0000 C CNN
-F 1 "Coil Pack" H 4450 6390 50  0000 C CNN
+F 0 "T2" H 4450 6481 50  0001 C CNN
+F 1 "Coil Pack 2" H 4450 6390 50  0000 C CNN
 F 2 "" H 4450 6100 50  0001 C CNN
 F 3 "~" H 4450 6100 50  0001 C CNN
@@
 U 1 1 6016E061
 P 4450 6750
-F 0 "T3" H 4450 7131 50  0000 C CNN
-F 1 "Coil Pack" H 4450 7040 50  0000 C CNN
+F 0 "T3" H 4450 7131 50  0001 C CNN
+F 1 "Coil Pack 3" H 4450 7040 50  0000 C CNN
 F 2 "" H 4450 6750 50  0001 C CNN
 F 3 "~" H 4450 6750 50  0001 C CNN
@@
 U 1 1 6016E079
 P 4450 7400
-F 0 "T4" H 4450 7781 50  0000 C CNN
-F 1 "Coil Pack" H 4450 7690 50  0000 C CNN
+F 0 "T4" H 4450 7781 50  0001 C CNN
+F 1 "Coil Pack 4" H 4450 7690 50  0000 C CNN
 F 2 "" H 4450 7400 50  0001 C CNN
 F 3 "~" H 4450 7400 50  0001 C CNN
@@
 L Switch:SW_DIP_x01 SW1
 U 1 1 601E11AA
-P 6050 6200
-F 0 "SW1" H 6050 6467 50  0000 C CNN
-F 1 "UPSHIFT" H 6050 6376 50  0000 C CNN
-F 2 "" H 6050 6200 50  0001 C CNN
-F 3 "~" H 6050 6200 50  0001 C CNN
-	1    6050 6200
+P 6100 6150
+F 0 "SW1" H 6100 6417 50  0000 C CNN
+F 1 "UPSHIFT" H 6100 6326 50  0000 C CNN
+F 2 "" H 6100 6150 50  0001 C CNN
+F 3 "~" H 6100 6150 50  0001 C CNN
+	1    6100 6150
 	1    0    0    -1
 $EndComp
@@
 L Switch:SW_DIP_x01 SW2
 U 1 1 601E11B4
-P 6050 6650
-F 0 "SW2" H 6050 6917 50  0000 C CNN
-F 1 "DOWNSHIFT" H 6050 6826 50  0000 C CNN
-F 2 "" H 6050 6650 50  0001 C CNN
-F 3 "~" H 6050 6650 50  0001 C CNN
-	1    6050 6650
+P 6100 6600
+F 0 "SW2" H 6100 6867 50  0000 C CNN
+F 1 "DOWNSHIFT" H 6100 6776 50  0000 C CNN
+F 2 "" H 6100 6600 50  0001 C CNN
+F 3 "~" H 6100 6600 50  0001 C CNN
+	1    6100 6600
 	1    0    0    -1
 $EndComp
@@
 L Switch:SW_DIP_x01 SW3
 U 1 1 601E11BE
-P 6050 7100
-F 0 "SW3" H 6050 7367 50  0000 C CNN
-F 1 "NEUTRAL" H 6050 7276 50  0000 C CNN
-F 2 "" H 6050 7100 50  0001 C CNN
-F 3 "~" H 6050 7100 50  0001 C CNN
-	1    6050 7100
+P 6100 7050
+F 0 "SW3" H 6100 7317 50  0000 C CNN
+F 1 "NEUTRAL" H 6100 7226 50  0000 C CNN
+F 2 "" H 6100 7050 50  0001 C CNN
+F 3 "~" H 6100 7050 50  0001 C CNN
+	1    6100 7050
 	1    0    0    -1
 $EndComp
@@
 L Switch:SW_DIP_x01 SW4
 U 1 1 601EA861
-P 6050 7550
-F 0 "SW4" H 6050 7817 50  0000 C CNN
-F 1 "START" H 6050 7726 50  0000 C CNN
-F 2 "" H 6050 7550 50  0001 C CNN
-F 3 "~" H 6050 7550 50  0001 C CNN
-	1    6050 7550
+P 6100 7500
+F 0 "SW4" H 6100 7767 50  0000 C CNN
+F 1 "START" H 6100 7676 50  0000 C CNN
+F 2 "" H 6100 7500 50  0001 C CNN
+F 3 "~" H 6100 7500 50  0001 C CNN
+	1    6100 7500
 	1    0    0    -1
 $EndComp
@@
 Text GLabel 7300 5900 0    50   Input ~ 0
 CANL
-Text Notes 3650 2950 0    50   ~ 0
+Text Notes 3750 2850 0    50   ~ 0
 Engine
 Text GLabel 2750 6100 0    50   Input ~ 0
@@
 U 1 1 60134F69
 P 6150 4550
-F 0 "U12" H 6150 4665 50  0000 C CNN
+F 0 "U12" H 6150 4665 50  0001 C CNN
 F 1 "WirelessTelemetry" H 6150 4574 50  0000 C CNN
 F 2 "" H 6150 4550 50  0001 C CNN
@@
 	1    0    0    -1
 $EndComp
-Wire Notes Line
-	2450 4900 2450 2950
 Wire Notes Line
 	5300 7750 5300 5000
@@
 U 1 1 6012B145
 P 3150 5900
-F 0 "U7" H 3125 6015 50  0000 C CNN
+F 0 "U7" H 3125 6015 50  0001 C CNN
 F 1 "BOSCH_W0133-1605554" H 3125 5924 50  0000 C CNN
 F 2 "" H 3150 5900 50  0001 C CNN
@@
 	1    0    0    -1
 $EndComp
-Wire Notes Line
-	8050 550  8050 1850
 Text Notes 7000 550  0    50   ~ 0
 Electronic Throttle Body
@@
 Text GLabel 8600 950  0    50   Input ~ 0
 BRAKEPRES
-Text GLabel 6350 6200 2    50   Input ~ 0
+Text GLabel 6400 6150 2    50   Input ~ 0
 UPSHIFT
 Text GLabel 9950 2000 0    50   Input ~ 0
@@
 Text GLabel 9950 2400 0    50   Input ~ 0
 DOWNSHIFT
-Text GLabel 6350 6650 2    50   Input ~ 0
+Text GLabel 6400 6600 2    50   Input ~ 0
 DOWNSHIFT
 Text GLabel 9950 2500 0    50   Input ~ 0
 NEUTRAL
-Text GLabel 6350 7100 2    50   Input ~ 0
+Text GLabel 6400 7050 2    50   Input ~ 0
 NEUTRAL
 Text GLabel 9950 2900 0    50   Input ~ 0
 START
-Text GLabel 6350 7550 2    50   Input ~ 0
+Text GLabel 6400 7500 2    50   Input ~ 0
 START
 Wire Notes Line
@@
 NoConn ~ 9400 800
 Wire Notes Line
-	11150 1700 11150 700
-Wire Notes Line
-	11150 700  9600 700
-Wire Notes Line
-	9600 700  9600 1700
-Wire Notes Line
-	9600 1700 11150 1700
-Wire Notes Line
 	11150 6500 9400 6500
 Wire Notes Line
@@
 +12v
 Wire Notes Line
-	9350 6500 7000 6500
-Wire Notes Line
 	6750 4200 8700 4200
 Wire Notes Line
@@
 	9300 4700 8400 4700
 Wire Notes Line
-	9350 4300 7000 4300
-Wire Notes Line
-	7000 4300 7000 6500
-Wire Notes Line
 	9350 4300 9350 6500
 Text GLabel 5750 4700 0    50   Input ~ 0
 +12v
 Wire Notes Line
-	5300 4900 5300 2950
-Wire Notes Line
-	2450 2950 5300 2950
-Wire Notes Line
 	2450 4900 5300 4900
 Wire Notes Line
@@
 Text Notes 5800 4300 0    50   ~ 0
 Wireless Telemetry
-Wire Notes Line
-	6650 550  6650 1850
-Wire Notes Line
-	6650 1850 8050 1850
 Wire Notes Line
 	6650 550  8050 550
@@
 NoConn ~ 1850 6850
 NoConn ~ 1850 6750
-Text GLabel 5650 6900 0    50   Input ~ 0
+Text GLabel 5700 6850 0    50   Input ~ 0
 +12v
 Wire Wire Line
-	5750 6200 5750 6650
-Connection ~ 5750 6650
-Wire Wire Line
-	5750 6650 5750 6900
-Connection ~ 5750 7100
-Wire Wire Line
-	5750 7100 5750 7550
-Wire Wire Line
-	5650 6900 5750 6900
-Connection ~ 5750 6900
-Wire Wire Line
-	5750 6900 5750 7100
+	5800 6150 5800 6600
+Connection ~ 5800 6600
+Wire Wire Line
+	5800 6600 5800 6850
+Connection ~ 5800 7050
+Wire Wire Line
+	5800 7050 5800 7500
+Wire Wire Line
+	5700 6850 5800 6850
+Connection ~ 5800 6850
+Wire Wire Line
+	5800 6850 5800 7050
 Text GLabel 1850 3300 2    50   Input ~ 0
 FUELPRES
@@
 Text GLabel 6250 3350 1    50   Input ~ 0
 RADFAN2
-Text GLabel 7550 2250 0    50   Input ~ 0
+Text GLabel 7500 2250 0    50   Input ~ 0
 BRAKELIGHT
 $Comp
 L Device:LED D1
 U 1 1 601A0AD2
-P 8000 2250
-F 0 "D1" H 8000 2050 50  0000 C CNN
-F 1 "LED" H 8000 2150 50  0000 C CNN
-F 2 "" H 8000 2250 50  0001 C CNN
-F 3 "~" H 8000 2250 50  0001 C CNN
-	1    8000 2250
+P 7950 2250
+F 0 "D1" H 7950 2050 50  0000 C CNN
+F 1 "LED" H 7950 2150 50  0000 C CNN
+F 2 "" H 7950 2250 50  0001 C CNN
+F 3 "~" H 7950 2250 50  0001 C CNN
+	1    7950 2250
 	-1   0    0    -1
 $EndComp
@@
 L Device:R_US R1
 U 1 1 601A0ADC
-P 7700 2250
-F 0 "R1" V 7900 2250 50  0000 C CNN
-F 1 "220" V 7800 2250 50  0000 C CNN
-F 2 "" V 7740 2240 50  0001 C CNN
-F 3 "~" H 7700 2250 50  0001 C CNN
-	1    7700 2250
+P 7650 2250
+F 0 "R1" V 7850 2250 50  0000 C CNN
+F 1 "220" V 7750 2250 50  0000 C CNN
+F 2 "" V 7690 2240 50  0001 C CNN
+F 3 "~" H 7650 2250 50  0001 C CNN
+	1    7650 2250
 	0    -1   1    0
 $EndComp
-Text Notes 7950 2150 2    50   ~ 0
+Text Notes 7900 2150 2    50   ~ 0
 Brake Light
 $Comp
 L power:GND #PWR021
 U 1 1 601A8EB9
-P 8300 2350
-F 0 "#PWR021" H 8300 2100 50  0001 C CNN
-F 1 "GND" H 8300 2200 50  0000 C CNN
-F 2 "" H 8300 2350 50  0001 C CNN
-F 3 "" H 8300 2350 50  0001 C CNN
-	1    8300 2350
-	1    0    0    -1
-$EndComp
-Wire Wire Line
-	8150 2250 8300 2250
-Wire Wire Line
-	8300 2250 8300 2350
-Wire Notes Line
-	8400 2550 8400 2150
-Wire Notes Line
-	8400 2150 7000 2150
-Wire Notes Line
-	7000 2150 7000 2550
-Wire Notes Line
-	7000 2550 8400 2550
-Wire Notes Line
-	8100 1850 9500 1850
+P 8250 2350
+F 0 "#PWR021" H 8250 2100 50  0001 C CNN
+F 1 "GND" H 8250 2200 50  0000 C CNN
+F 2 "" H 8250 2350 50  0001 C CNN
+F 3 "" H 8250 2350 50  0001 C CNN
+	1    8250 2350
+	1    0    0    -1
+$EndComp
+Wire Wire Line
+	8100 2250 8250 2250
+Wire Wire Line
+	8250 2250 8250 2350
+Wire Notes Line
+	8350 2550 8350 2150
+Wire Notes Line
+	8350 2150 6950 2150
+Wire Notes Line
+	6950 2150 6950 2550
+Wire Notes Line
+	6950 2550 8350 2550
 Text Notes 8200 550  0    50   ~ 0
 Brake System Plausability Device
 Wire Notes Line
 	9500 550  8100 550
-Wire Notes Line
-	8100 550  8100 1850
-Wire Notes Line
-	9500 550  9500 1850
 Text Notes 4100 550  0    50   ~ 0
 Power Management Unit
@@
 NoConn ~ 1850 3900
 NoConn ~ 1850 3400
+Wire Notes Line
+	9550 550  11150 550
+Wire Notes Line
+	9550 550  9550 1800
+Wire Notes Line
+	9550 1800 11150 1800
+Wire Notes Line
+	11150 1800 11150 550
+Wire Notes Line
+	9500 550  9500 1800
+Wire Notes Line
+	9500 1800 8100 1800
+Wire Notes Line
+	8100 1800 8100 550
+Wire Notes Line
+	8050 550  8050 1800
+Wire Notes Line
+	8050 1800 6650 1800
+Wire Notes Line
+	6650 1800 6650 550
+Wire Notes Line
+	5300 2850 2450 2850
+Wire Notes Line
+	2450 2850 2450 4900
+Wire Notes Line
+	5300 2850 5300 4900
+Wire Notes Line
+	6950 4300 6950 6500
+Wire Notes Line
+	6950 6500 9350 6500
+Wire Notes Line
+	6950 4300 9350 4300
+Wire Wire Line
+	5000 1700 5000 1800
+Wire Wire Line
+	5000 1800 4950 1800
+Wire Wire Line
+	4950 1800 4950 1900
 $EndSCHEMATC
